Commit message: fixed dimmensions

File: description/lidar.xacro (robot description, xacro)
@@ -4,5 +4,5 @@
         <parent link="chassis"/>
         <child link="laser_frame"/>
-        <origin xyz="0.1 0 0.06" rpy="0 0 0"/>
+        <origin xyz="0.25 0 0.06" rpy="0 0 0"/>
     </joint>
     <link name="laser_frame">

File: description/robot_core.xacro (robot description, xacro)
@@ -30,5 +30,5 @@
     <link name="chassis">
         <visual>
-            <origin xyz="0.15 0.0 0.01"/>
+            <origin xyz="0.15 0.0 0.02"/>
             <geometry>
                 <cylinder radius="0.17" length="0.06"/>
@@ -58,5 +58,5 @@
         <visual>
             <geometry>
-                <cylinder radius="0.03" length="0.04"/>
+                <cylinder radius="0.022" length="0.02"/>
             </geometry>
             <material name="blue"></material>
@@ -64,8 +64,8 @@
         <collision>
             <geometry>
-                <cylinder radius="0.03" length="0.04"/>
+                <cylinder radius="0.03" length="0.02"/>
             </geometry>
         </collision>
-        <xacro:inertial_cylinder mass="0.1" radius="0.03" length="0.04">
+        <xacro:inertial_cylinder mass="0.1" radius="0.022" length="0.02">
             <origin xyz="0.0 0.0 0.0" rpy="0.0 0.0 0.0"/>
         </xacro:inertial_cylinder>
@@ -83,5 +83,5 @@
         <visual>
             <geometry>
-                <cylinder radius="0.03" length="0.04"/>
+                <cylinder radius="0.022" length="0.02"/>
             </geometry>
             <material name="blue"></material>
@@ -89,5 +89,5 @@
         <collision>
             <geometry>
-                <cylinder radius="0.03" length="0.04"/>
+                <cylinder radius="0.022" length="0.02"/>
             </geometry>
         </collision>
@@ -107,5 +107,5 @@
         <visual>
             <geometry>
-                <sphere radius="0.02"/>
+                <sphere radius="0.01"/>
             </geometry>
             <material name="black"></material>
@@ -113,8 +113,8 @@
         <collision>
             <geometry>
-                <sphere radius="0.02"/>
+                <sphere radius="0.01"/>
             </geometry>
         </collision>
-        <xacro:inertial_sphere mass="0.1" radius="0.02">
+        <xacro:inertial_sphere mass="0.1" radius="0.01">
             <origin xyz="0.0 0.0 0.0" rpy="0.0 0.0 0.0"/>
         </xacro:inertial_sphere>
